Commit message: a

File: description/robot.urdf.xacro (robot description, xacro)
@@ -2,4 +2,6 @@
 <robot xmlns:xacro="http://www.ros.org/wiki/xacro"  name="robot">
     <xacro:include filename="robot_core.xacro" />
-    <xacro:include filename="gazebo_control.xacro" />
+   <!-- <xacro:include filename="gazebo_control.xacro" />-->
+    <xacro:include filename="lidar.xacro" />
+    <xacro:include filename="ros2_control.xacro" />
 </robot>

File: description/robot_core.xacro (robot description, xacro)
@@ -19,9 +19,9 @@
     <parent link="base_link"/>
     <child link="chassis"/>
-    <origin xyz="-0.07 0 0"/>
+    <origin xyz="-0.07 0 0.06"/>
     </joint>
     <link name="chassis">
     <visual>
-        <origin xyz="0.28 0 0.35" rpy="0 0 0"/>
+        <origin xyz="0.28 0 0.41" rpy="0 0 0"/>
         <geometry>
             <cylinder length="0.7" radius="0.275"/>
@@ -30,5 +30,5 @@
     </visual>
     <collision>
-        <origin xyz="0.28 0 0.35" rpy="0 0 0"/>
+        <origin xyz="0.28 0 0.41" rpy="0 0 0"/>
         <geometry>
             <cylinder length="0.7" radius="0.275"/>
@@ -46,5 +46,5 @@
     <parent link="base_link"/>
     <child link="left_wheel"/>
-    <origin xyz="0 0.28 0" rpy="-${pi/2} 0 0"/>
+    <origin xyz="0 0.28 0.06" rpy="-${pi/2} 0 0"/>
     <axis xyz="0 0 1"/>
     </joint>
@@ -73,5 +73,5 @@
     <parent link="base_link"/>
     <child link="right_wheel"/>
-    <origin xyz="0 -0.28 0" rpy="${pi/2} 0 0"/>
+    <origin xyz="0 -0.28 0.06" rpy="${pi/2} 0 0"/>
     <axis xyz="0 0 -1"/>
     </joint>
@@ -100,10 +100,10 @@
     <parent link="chassis"/>
     <child link="caster_wheel"/>
-    <origin xyz="0.45 0 0" rpy="0 0 0"/>
+    <origin xyz="0.45 0 0" rpy="${pi/2} 0 0"/>
     </joint>
     <link name="caster_wheel">
     <visual>
         <geometry>
-            <sphere radius="0.085" />
+            <cylinder length="0.04" radius="0.065" />/>
         </geometry>
         <material name="blue"/>
@@ -111,11 +111,11 @@
     <collision>
         <geometry>
-            <sphere radius="0.085" />
+            <cylinder length="0.04" radius="0.065" />/>
         </geometry>
         <material name="blue"/>
     </collision>
-    <xacro:inertial_sphere mass="0.1" radius="0.085">
+    <xacro:inertial_cylinder mass="0.1" length="0.04" radius="0.065">
         <origin xyz="0 0 0" rpy="0 0 0"/>
-    </xacro:inertial_sphere>
+    </xacro:inertial_cylinder>
     </link>
     <gazebo reference="caster_wheel">
